File: attinyProgrammer/attinyProgrammer.kicad_pcb (KiCad board)
At the start: 4 copper layers, 50 x 20 mm, 30 parts, among them J1 USB_C_Receptacle_USB2.0_16P, J4 Conn_02x06_Odd_Even, SW1 SW_SPST, U1 STM32F042K6Tx, U2 24LC64, U3 MT3608, U4 AMS1117-3.3, U5 USBLC6-2SC6

Commit message: Semi-Final PCB, waiting on last touches and then to order
Parts:
- removed C8: 10u, Capacitor_SMD:C_0603_1608Metric_Pad1.08x0.95mm_HandSolder
- removed C9: 22u, Capacitor_SMD:C_0603_1608Metric_Pad1.08x0.95mm_HandSolder
- removed U4: AMS1117-3.3, Package_TO_SOT_SMD:SOT-223-3_TabPin2
- added D2: LED, LED_SMD:LED_0603_1608Metric_Pad1.05x0.95mm_HandSolder, F.Cu at (122.2, 81.8)
- added R7: 4.7k, Resistor_SMD:R_0603_1608Metric_Pad0.98x0.95mm_HandSolder, F.Cu at (132.2, 87.8)
- added R8: 4.7k, Resistor_SMD:R_0603_1608Metric_Pad0.98x0.95mm_HandSolder, F.Cu at (138.2, 86.0)
- added R9: 4.7k, Resistor_SMD:R_0603_1608Metric_Pad0.98x0.95mm_HandSolder, F.Cu at (120.0, 81.8)
- added U6: 74AHCT1G08, PCM_SparkFun-Semiconductor-Standard:SOT23-5, B.Cu at (122.0, 94.5)
- added U7: 74AHCT1G08, PCM_SparkFun-Semiconductor-Standard:SOT23-5, B.Cu at (132.2, 91.5)
- added U8: 74AHCT1G08, PCM_SparkFun-Semiconductor-Standard:SOT23-5, B.Cu at (127.5, 94.5)
- C2: moved to B.Cu
- U3: moved to F.Cu
- moved C2 55.6 mm to (118.5, 95.2), turned to 90 degrees
- moved U3 44.8 mm to (170.0, 86.0), turned to 180 degrees
- moved C13 24.4 mm to (184.0, 82.2)
- moved L1 24.4 mm to (184.0, 84.8)
- moved R6 24.4 mm to (184.0, 89.8)
- moved C12 24.4 mm to (184.0, 79.7)
- moved R5 24.4 mm to (184.0, 87.3)
- moved SW1 13.9 mm to (109.0, 94.0)
- moved D1 12.4 mm to (176.8, 81.8)
- moved C3 2.77 mm to (134.8, 87.0), turned to 0 degrees
- moved C4 1.03 mm to (132.8, 94.2), turned to 0 degrees
- moved C11 0.75 mm to (114.0, 82.0)
- moved C6 0.75 mm to (138.5, 82.0), turned to 90 degrees
Connections:
- J4 pad 1: unconnected-(J4-Pin_1-Pad1) -> USART_RX
- J4 pad 10: unconnected-(J4-Pin_10-Pad10) -> TPIDATA // SPI
- J4 pad 11: unconnected-(J4-Pin_11-Pad11) -> SWCLK
- J4 pad 12: unconnected-(J4-Pin_12-Pad12) -> TPICLK // SPI_SCK
- J4 pad 2: TPICLK // SPI_SCK -> USART_TX
- J4 pad 3: unconnected-(J4-Pin_3-Pad3) -> PB8
- J4 pad 4: unconnected-(J4-Pin_4-Pad4) -> GND
- J4 pad 5: unconnected-(J4-Pin_5-Pad5) -> +3.3V
- J4 pad 6: unconnected-(J4-Pin_6-Pad6) -> +5V
- J4 pad 8: unconnected-(J4-Pin_8-Pad8) -> RESET // GPIO
- J4 pad 9: unconnected-(J4-Pin_9-Pad9) -> SWDIO
- U1 pad 10: unconnected-(U1-PA4-Pad10) -> RESET // GPIO
- U1 pad 12: SPI_MISO -> unconnected-(U1-PA6-Pad12)
- U1 pad 19: unconnected-(U1-PA9-Pad19) -> USART_TX
- U1 pad 20: unconnected-(U1-PA10-Pad20) -> USART_RX
- U1 pad 23: unconnected-(U1-PA13-Pad23) -> SWDIO
- U1 pad 24: unconnected-(U1-PA14-Pad24) -> SWCLK
- U1 pad 31: unconnected-(U1-PB8-Pad31) -> PB8
- U1 pad 9: unconnected-(U1-PA3-Pad9) -> TPIDATA // SPI
Routing:
- net +3.3V: track 13.1 -> 99.7 mm, vias 0 -> 7
- net +5V: track 17.4 -> 89.1 mm, vias 1 -> 5
- net SWDIO: track 0.00 -> 46.3 mm
- net SWCLK: track 0.00 -> 40.9 mm
- net USART_RX: track 0.00 -> 38.1 mm, vias 0 -> 1
- net PB8: track 0.00 -> 32.1 mm
- net USART_TX: track 0.00 -> 31.7 mm, vias 0 -> 1
- net Net-(SW1-B): track 0.00 -> 28.1 mm, vias 0 -> 1
- net TPIDATA // SPI: track 0.00 -> 25.8 mm, vias 0 -> 1
- net GND: track 28.1 -> 52.7 mm, vias 12 -> 20
- net RESET // GPIO: track 0.00 -> 18.8 mm, vias 0 -> 1
- net TPICLK // SPI_SCK: track 19.5 -> 31.2 mm
- net Net-(D2-A): track 0.00 -> 2.27 mm
- net EEPROM_SCLK: track 14.1 -> 16.1 mm
- net EEPROM_SDA: track 14.2 -> 16.2 mm
Other:
- board text added: "+5V"
- board text added: "PB8"
- board text added: "RX"
- board text added: "TPICLK"
- board text added: "TPIRESET"
- board text added: "TX"
