File: attinyProgrammer/attinyProgrammer.kicad_sch (KiCad schematic)
At the start: 30 parts, among them J1 USB_C_Receptacle_USB2.0_16P, J4 Conn_02x06_Odd_Even, SW1 SW_SPST, U1 STM32F042K6Tx, U2 24LC64, U3 MT3608, U4 AMS1117-3.3, U5 USBLC6-2SC6

Commit message: Semi-Final PCB, waiting on last touches and then to order
Parts:
- removed C8: 10u, Capacitor_SMD:C_0603_1608Metric_Pad1.08x0.95mm_HandSolder, symbol Device:C
- removed C9: 22u, Capacitor_SMD:C_0603_1608Metric_Pad1.08x0.95mm_HandSolder, symbol Device:C
- removed U4: AMS1117-3.3, Package_TO_SOT_SMD:SOT-223-3_TabPin2, symbol Regulator_Linear:AMS1117-3.3
- added D2: LED, LED_SMD:LED_0603_1608Metric_Pad1.05x0.95mm_HandSolder, symbol Device:LED
- added R7, R8, R9: 4.7k, Resistor_SMD:R_0603_1608Metric_Pad0.98x0.95mm_HandSolder, symbol Device:R
- added U6, U7, U8: 74AHCT1G08, PCM_SparkFun-Semiconductor-Standard:SOT23-5, symbol 74xGxx:74AHCT1G08
Connections:
- net +3.3V: now also J4.5 (Pin_5), R7.1, R8.1, R9.1
- net +5V: now also J4.6 (Pin_6), U6.1, U6.5 (VCC), U7.1, U7.5 (VCC), U8.1, U8.5 (VCC)
- net EEPROM_SCLK: now also R7.2
- net EEPROM_SDA: now also R8.2
- net GND: now also J4.4 (Pin_4), D2.1 (K), U6.3 (GND), U7.3 (GND), U8.3 (GND)
- net RESET // GPIO: now also J4.8 (Pin_8), U1.10 (PA4), U7.2, U7.4
- net SWCLK: now also J4.11 (Pin_11), U1.24 (PA14)
- net SWDIO: now also J4.9 (Pin_9), U1.23 (PA13)
- net TPICLK // SPI_SCK: now also J4.12 (Pin_12), U6.2, U6.4; no longer J4.2 (Pin_2)
- net USART_RX: now reaches J4.1 (Pin_1)
- net USART_RX: now also U1.20 (PA10)
- net TPIDATA // SPI: now reaches J4.10 (Pin_10)
- net TPIDATA // SPI: now also U1.9 (PA3), U8.2, U8.4
- net PB8: now reaches J4.3 (Pin_3)
- net PB8: now also U1.31 (PB8)
- net USART_TX: now reaches U1.19 (PA9)
- net USART_TX: now also J4.2 (Pin_2)
- net SPI_MISO: no longer names the net of U1.12 (PA6)
- new net: D2.2 (A), R9.2
Other:
- note removed: "5V -> 3.3V"
